Commit message: Add full paddle

File: ball_and_paddle.urdf (robot description, URDF)
Before this commit: robot BallAndPaddle, 2 links, 1 joints
Links:
- removed link paddle
- added link paddle_handle, mass .008; visual cylinder length=.1 radius=.013
- added link paddle_head, mass .042; visual cylinder length=.016 radius=.08
- link ball: mass .001 -> .0027; geometry visual sphere radius=0.02
Joints:
- joint paddle_fixed: child paddle -> paddle_head; origin xyz=0 0 -.0025 rpy=0 0 0 -> xyz=0 0 .09 rpy=1.5707963268 0 0; parent world -> paddle_handle

Commit message: Parameterize urdf

File: ball_and_paddle.urdf (robot description, URDF)
Before this commit: robot BallAndPaddle, 3 links, 1 joints
Links:
- added link table; visual box size=${table.wx} ${table.wy} ${table.wz}
- added link wall; visual box size=${wall.wx} ${wall.wy} ${wall.wz}
- link ball: mass .0027 -> ${ball.m}; geometry visual sphere radius=${ball.r}
- link paddle_handle: mass .008 -> ${handle.m}; geometry visual cylinder length=${handle.l} radius=${handle.r}
- link paddle_head: mass .042 -> ${head.m}; geometry visual cylinder length=${head.l} radius=${head.r}
Joints:
- added joint table_fixed: type fixed, parent world, child table, origin xyz=${table.x} ${table.y} ${table.z}
- added joint wall_fixed: type fixed, parent table, child wall, origin xyz=0 ${wall.yoffset} ${wall.zoffset}
- joint paddle_fixed: origin xyz=0 0 .09 rpy=1.5707963268 0 0 -> xyz=0 0 ${head.zoffset} rpy=${hpi} 0 0

Commit message: remove table and wall

File: ball_and_paddle.urdf (robot description, URDF)
Before this commit: robot BallAndPaddle, 5 links, 3 joints
Links:
- removed link table
- removed link wall
Joints:
- removed joint table_fixed
- removed joint wall_fixed

Commit message: remove ball

File: ball_and_paddle.urdf (robot description, URDF)
Before this commit: robot BallAndPaddle, 3 links, 1 joints
Links:
- removed link ball

Commit message: add ball back

File: ball_and_paddle.urdf (robot description, URDF)
Before this commit: robot BallAndPaddle, 2 links, 1 joints
Links:
- added link ball, mass ${ball.m}; visual sphere radius=${ball.r}

Commit message: lock ball

File: ball_and_paddle.urdf (robot description, URDF)
Before this commit: robot BallAndPaddle, 3 links, 1 joints
Joints:
- added joint ball_fixed: type fixed, parent world, child ball

Commit message: prismatic ball

File: ball_and_paddle.urdf (robot description, URDF)
Before this commit: robot BallAndPaddle, 3 links, 2 joints
Joints:
- removed joint ball_fixed
- added joint ball_prismatic: type prismatic, parent world, child ball, axis 0 0 1

Commit message: paddle prismatic

File: ball_and_paddle.urdf (robot description, URDF)
Before this commit: robot BallAndPaddle, 3 links, 2 joints
Joints:
- added joint paddle_prismatic: type prismatic, parent world, child paddle_handle, axis 0 0 1

Commit message: remove prismatic

File: ball_and_paddle.urdf (robot description, URDF)
Before this commit: robot BallAndPaddle, 3 links, 3 joints
Joints:
- removed joint ball_prismatic
- removed joint paddle_prismatic

Commit message: add back table and wall

File: ball_and_paddle.urdf (robot description, URDF)
Before this commit: robot BallAndPaddle, 3 links, 1 joints
Links:
- added link table; visual box size=${table.wx} ${table.wy} ${table.wz}
- added link wall; visual box size=${wall.wx} ${wall.wy} ${wall.wz}
Joints:
- added joint table_fixed: type fixed, parent world, child table, origin xyz=${table.x} ${table.y} ${table.z}
- added joint wall_fixed: type fixed, parent table, child wall, origin xyz=0 ${wall.yoffset} ${wall.zoffset}
